File: pcb/Power.kicad_sch (KiCad schematic)
At the start: 89 parts, among them J5 Barrel_Jack_Switch, Q2 ZXMC3A16DN8, U1 LFE5U-85F-6BG381, U8 LTC4360-2, U9 LTM8051

Commit message: Fix typo in R43 (1.35V output selection) value
Parts:
- R43: value 375k -> 357k
Changed lines of the file:
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@@
     (in_bom yes) (on_board yes)
     (property "Reference" "R43" (id 0) (at 149.86 162.56 90))
-    (property "Value" "375k" (id 1) (at 149.86 167.64 90))
+    (property "Value" "357k" (id 1) (at 149.86 167.64 90))
     (property "Footprint" "Resistor_SMD:R_0402_1005Metric" (id 2) (at 150.114 164.084 90)
       (effects (font (size 1.27 1.27)) hide)
