File: pcb/ecp5u85-bse-usb.kicad_sch (KiCad schematic)
At the start: 16 parts, among them J1 BSE-040-01-X-D-A, J2 BSE-040-01-X-D-A

Commit message: Rev. A before fab comments
- Added gerbers, mount positions, etc.
Other:
- note removed: "Even pins 32-74 are not really used in the acq. board (32 & 34 for daisy chain conn. 74 to gnd. Others to breakout section) So they can be moved freely. If you change differential IO locations, make sure that swaps happen between I vs. IO types. I can be swapped with I and IO with IO but not between."
- moved on the sheet: D1, D2, D3, R10, R8, R9
