File: test-pcb/ecp5u85-bse-usb_io-tester.kicad_sch (KiCad schematic)
At the start: 65 parts, among them J1 BTE-040-02-L-D-A, J2 Conn_01x09_Male, J3 BTE-040-02-L-D-A, U1 74HCT4067PW,118, U10 74HCT4067PW,118, U2 74HCT4067PW,118, U3 NCV4274ADT33RKG, U4 74HCT4067PW,118, U5 74HCT4067PW,118, U6 ATxmega32A4U-A, U7 74HCT4067PW,118, U8 74HCT4067PW,118, U9 74HCT4067PW,118

Commit message: Initial completed IO test board
- Schematic and layout should be finished.
- Will generate gerbers upon approval
Parts:
- removed D4: LED, LED_SMD:LED_0603_1608Metric, symbol Device:LED
- removed J2: Conn_01x09_Male, Connector_PinHeader_2.54mm:PinHeader_1x10_P2.54mm_Horizontal, symbol Connector:Conn_01x09_Male
- removed R11: 1k, Resistor_SMD:R_0402_1005Metric, symbol Device:R_US
- added C13: 0.1uF, Capacitor_SMD:C_0402_1005Metric, symbol Device:C
- added C14, C17, C18, C19, C23, C24, C25: 0.1uF, Capacitor_SMD:C_0603_1608Metric, symbol Device:C
- added C15: 100uF, Capacitor_Tantalum_SMD:CP_EIA-6032-28_Kemet-C, symbol Device:C_Polarized
- added C16: 4.7uF, Capacitor_SMD:C_0805_2012Metric, symbol Device:C
- added C20, C21: 47pF, Capacitor_SMD:C_0603_1608Metric, symbol Device:C
- added C22: 4.7nF, Capacitor_SMD:C_0603_1608Metric, symbol Device:C
- added D6: LED, LED_SMD:LED_0603_1608Metric, symbol Device:LED
- added FB1: FerriteBead, Inductor_SMD:L_0603_1608Metric, symbol Device:FerriteBead
- added J2: USB_B_Mini, Connector_USB:USB_Mini-B_Lumberg_2486_01_Horizontal, symbol Connector:USB_B_Mini
- added J4: Conn_02x03_Odd_Even, Connector_PinHeader_2.54mm:PinHeader_2x03_P2.54mm_Vertical, symbol Connector_Generic:Conn_02x03_Odd_Even
- added J5: Conn_02x10_Odd_Even, Connector_PinHeader_2.54mm:PinHeader_2x10_P2.54mm_Vertical, symbol Connector_Generic:Conn_02x10_Odd_Even
- added L1: L, Inductor_SMD:L_1206_3216Metric, symbol Device:L
- added R15, R16, R17, R18, R20, R21, R22, R23: 1k, Resistor_SMD:R_0402_1005Metric, symbol Device:R_US
- added R19: 100, Resistor_SMD:R_0402_1005Metric, symbol Device:R_US
- added SW1: SW_Push, Button_Switch_THT:SW_PUSH_6mm_H8mm, symbol Switch:SW_Push
- added TP2: TestPoint, TestPoint:TestPoint_THTPad_3.0x3.0mm_Drill1.5mm, symbol Connector:TestPoint
- added U11: 74HCT4067PW,118, Package_SO:TSSOP-24_4.4x7.8mm_P0.65mm, symbol 74xx:CD74HC4067M
- added U12: FT232RL, Package_SO:SSOP-28_5.3x10.2mm_P0.65mm, symbol Interface_USB:FT232RL
- added U13: OSCILLATOR_EN, Oscillator:Oscillator_SMD_Abracon_ASE-4Pin_3.2x2.5mm, symbol jonnew:OSCILLATOR_EN
- TP1: footprint TestPoint:TestPoint_Plated_Hole_D2.0mm -> TestPoint:TestPoint_THTPad_3.0x3.0mm_Drill1.5mm
Connections:
- net Enable_{0} is gone; now on net +5V: U1.15 (~{E}), U2.15 (~{E}), U7.15 (~{E}), U8.15 (~{E})
- net Enable_{1} is gone; now on net +5V: U10.15 (~{E}), U4.15 (~{E}), U5.15 (~{E}), U9.15 (~{E})
- net +3V3: now also U6.19 (VCC), U6.31 (VCC), U6.9 (VCC), C18.1, C23.1, C25.1, FB1.2, J4.2 (Pin_2), R15.2, R20.2, TP2.1, U12.4 (VCCIO), U13.1 (EN), U13.4 (VCC); no longer U6.39 (AVCC)
- net +5V: now also C13.1, C15.1, C16.1, C17.1, L1.2, U11.15 (~{E}), U11.24 (VCC), U12.20 (VCC); no longer J1.1 (Pin_1), J1.3 (Pin_3), J1.5 (Pin_5)
- net A_{0}: now also U6.14 (PC4), U11.10 (S0)
- net A_{1}: now also U6.15 (PC5), U11.11 (S1)
- net A_{2}: now also U6.16 (PC6), U11.14 (S2)
- net A_{3}: now also U6.17 (PC7), U11.13 (S3)
- net D2I0+: now also U2.16 (I15); no longer U2.6 (I3)
- net D2I0-: now also U2.17 (I14); no longer U2.5 (I4)
- net D2I1+: now also U2.18 (I13); no longer U2.4 (I5)
- net D2I1-: now also U2.19 (I12); no longer U2.3 (I6)
- net D2I2+: now also U1.9 (I0); no longer U1.7 (I2)
- net D2I2-: now also U1.5 (I4); no longer U1.6 (I3)
- net D2I3+: now also U1.8 (I1); no longer U1.5 (I4)
- net D2I4+: now also U1.6 (I3); no longer U1.23 (I8)
- net D2I4-: now also U1.2 (I7); no longer U1.22 (I9)
- net D2IO0+: now also U5.19 (I12); no longer U5.4 (I5)
- net D2IO0-: now also U5.22 (I9); no longer U5.3 (I6)
- net D2IO1+: now also U5.21 (I10); no longer U5.2 (I7)
- net D2IO1-: now also U5.3 (I6); no longer U5.23 (I8)
- net D2IO2+: now also U5.23 (I8); no longer U5.22 (I9)
- net D2IO2-: now also U5.2 (I7); no longer U5.21 (I10)
- net D2IO4+: now also U2.20 (I11); no longer U2.2 (I7)
- net D2IO4-: now also U2.21 (I10); no longer U2.23 (I8)
- net D2IO5-: now also U4.22 (I9); no longer U4.2 (I7)
- net D2IO6-: now also U2.23 (I8); no longer U2.21 (I10)
- net D2IO7+: now also U2.3 (I6); no longer U2.20 (I11)
- net D2IO7-: now also U2.2 (I7); no longer U2.19 (I12)
- net D2IO8+: now also U5.4 (I5); no longer U5.20 (I11)
- net D2IO8-: now also U5.5 (I4); no longer U5.19 (I12)
- net D3I0+: now also U1.23 (I8); no longer U1.21 (I10)
- net D3I0-: now also U1.16 (I15); no longer U1.20 (I11)
- net D3I1+: now also U1.7 (I2); no longer U1.3 (I6)
- net D3I1-: now also U1.3 (I6); no longer U1.2 (I7)
- net D3I2+: now also U1.22 (I9); no longer U1.19 (I12)
- net D3I2-: now also U1.17 (I14); no longer U1.18 (I13)
- net D3I3+: now also U2.6 (I3); no longer U2.16 (I15)
- net D3I3-: now also U2.7 (I2); no longer U5.9 (I0)
- net D3I4+: now also U2.4 (I5); no longer U2.18 (I13)
- net D3I4-: now also U2.5 (I4); no longer U2.17 (I14)
- net D3I5+: now also U1.21 (I10); no longer U1.17 (I14)
- net D3I5-: now also U1.18 (I13); no longer U1.16 (I15)
- net D3I6+: now also U1.20 (I11); no longer U4.9 (I0)
- net D3I6-: now also U1.19 (I12); no longer U4.8 (I1)
- net D3I7-: now also U4.16 (I15); no longer U4.18 (I13)
- net D3IO0+: now also U2.8 (I1); no longer U5.8 (I1)
- net D3IO0-: now also U2.9 (I0); no longer U5.7 (I2)
- net D3IO1-: now also U4.21 (I10); no longer U4.22 (I9)
- net D3IO2+: now also U5.6 (I3); no longer U5.18 (I13)
- net D3IO2-: now also U5.7 (I2); no longer U5.17 (I14)
- net D3IO3+: now also U4.20 (I11); no longer U4.21 (I10)
- net D3IO3-: now also U4.17 (I14); no longer U4.20 (I11)
- net D3IO4+: now also U5.18 (I13); no longer U5.6 (I3)
- net D3IO4-: now also U5.20 (I11); no longer U5.5 (I4)
- net D3IO6+: now also U5.9 (I0); no longer U10.16 (I15)
- net D3IO7+: now also U4.18 (I13); no longer U4.17 (I14)
- net D3IO7-: now also U5.8 (I1); no longer U5.16 (I15)
- net D6I0+: now also U8.21 (I10); no longer U8.23 (I8)
- net D6I0-: now also U8.6 (I3); no longer U8.22 (I9)
- net D6I1+: now also U8.16 (I15); no longer U8.9 (I0)
- net D6I1-: now also U8.17 (I14); no longer U8.8 (I1)
- net D6I2+: now also U8.23 (I8); no longer U8.7 (I2)
- net D6I2-: now also U8.18 (I13); no longer U8.6 (I3)
- net D6I3+: now also U8.2 (I7); no longer U8.3 (I6)
- net D6I3-: now also U8.20 (I11); no longer U8.2 (I7)
- net D6I4+: now also U9.3 (I6); no longer U9.2 (I7)
- net D6I4-: now also U9.21 (I10); no longer U9.23 (I8)
- net D6I5+: now also U8.22 (I9); no longer U8.5 (I4)
- net D6I5-: now also U8.19 (I12); no longer U8.4 (I5)
- net D6I6+: now also U9.5 (I4); no longer U9.6 (I3)
- net D6I6-: now also U9.6 (I3); no longer U9.5 (I4)
- net D6I7-: now also U9.2 (I7); no longer U9.3 (I6)
- net D6IO0+: now also U7.5 (I4); no longer U7.6 (I3)
- net D6IO0-: now also U7.4 (I5); no longer U7.5 (I4)
- net D6IO1+: now also U7.3 (I6); no longer U7.4 (I5)
- net D6IO1-: now also U7.2 (I7); no longer U7.3 (I6)
- net D6IO3+: now also U7.6 (I3); no longer U7.2 (I7)
- net D6IO3-: now also U7.7 (I2); no longer U7.23 (I8)
- net D6IO4+: now also U7.23 (I8); no longer U7.20 (I11)
- net D6IO5+: now also U7.21 (I10); no longer U7.22 (I9)
- net D6IO5-: now also U7.22 (I9); no longer U7.21 (I10)
- net GND: now also R14.1, R8.1, U10.2 (I7), U4.2 (I7), U4.8 (I1), U4.9 (I0), U5.16 (I15), U5.17 (I14), U6.18 (GND), U6.30 (GND), U6.38 (GND), U6.8 (GND), U7.20 (I11), U7.8 (I1), U7.9 (I0), C13.2, C14.2, C15.2, C16.2, C17.2, C18.2, C19.2, C20.2, C21.2, C22.2, C23.2, C24.2, C25.2, D6.1 (K), J2.5 (GND), J4.6 (Pin_6), J5.10 (Pin_10), J5.12 (Pin_12), J5.14 (Pin_14), J5.16 (Pin_16), J5.18 (Pin_18), J5.2 (Pin_2), J5.20 (Pin_20), J5.4 (Pin_4), J5.6 (Pin_6), J5.8 (Pin_8), R17.1, R19.1, SW1.2, U11.12 (GND), U11.16 (I15), U11.17 (I14), U11.2 (I7), U11.20 (I11), U12.18 (GND), U12.21 (GND), U12.25 (AGND), U12.26 (TEST), U12.7 (GND), U13.2 (GND)
- net J1-11_3.3V: now also R5.1, U11.8 (I1); no longer J1.11 (Pin_11), R5.2
- net J1-13_3.3V: now also R6.1, U11.9 (I0); no longer J1.13 (Pin_13), R6.2
- net J1-4_RAMVDD: now also R1.2, U11.23 (I8); no longer J1.4 (Pin_4), R1.1
- net J1-6_RAMVDD: now also R2.2, U11.22 (I9); no longer J1.6 (Pin_6), R2.1
- net J1-7_2.5V: now also R3.1, U11.3 (I6); no longer J1.7 (Pin_7), R3.2
- net J1-9_3.3V: now also R4.1, U11.7 (I2); no longer J1.9 (Pin_9), R4.2
- net J2-2_3.3V: now also R21.2, U11.21 (I10); no longer J3.2 (Pin_2), R8.1
- net J2-4_3.3V: now also R22.2, U11.19 (I12); no longer J3.4 (Pin_4), R13.1
- net J2-6_3.3V: now also R23.2, U11.18 (I13); no longer J3.6 (Pin_6), R14.1
- net RX: now also U6.33 (PE3), U12.5 (RXD)
- net S00: now also U10.21 (I10); no longer U10.7 (I2)
- net S01: now also U10.19 (I12); no longer U10.4 (I5)
- net S02: now also U10.22 (I9); no longer U10.5 (I4)
- net S03: now also U10.16 (I15); no longer U10.9 (I0)
- net S04: now also U10.18 (I13); no longer U10.6 (I3)
- net S05: now also U8.9 (I0); no longer U8.16 (I15)
- net S06: now also U10.17 (I14); no longer U10.8 (I1)
- net S07: now also U10.23 (I8); no longer U10.3 (I6)
- net S10: now also U10.6 (I3); no longer U10.22 (I9)
- net S11: now also U9.23 (I8); no longer U9.21 (I10)
- net S111: now also U10.5 (I4); no longer U10.23 (I8)
- net S13: now also U8.8 (I1); no longer U8.18 (I13)
- net S14: now also U8.5 (I4); no longer U8.17 (I14)
- net S15: now also U10.8 (I1); no longer U10.18 (I13)
- net S17: now also U10.20 (I11); no longer U10.2 (I7)
- net S19: now also U10.7 (I2); no longer U10.20 (I11)
- net S60: now also U8.3 (I6); no longer U8.21 (I10)
- net S81: now also U10.3 (I6); no longer U10.21 (I10)
- net S83: now also U10.9 (I0); no longer U10.17 (I14)
- net S84: now also U8.4 (I5); no longer U8.19 (I12)
- net S85: now also U10.4 (I5); no longer U10.19 (I12)
- net S86: now also U8.7 (I2); no longer U8.20 (I11)
- net TX: now also U6.32 (PE2), U12.1 (TXD)
- net TestClock: now also U6.10 (PC0), J5.19 (Pin_19)
- net at R12.2: now also U6.36 (PR0/XTAL2)
- net at R10.2: now also U6.24 (PD4)
- net J1-3_5V: now reaches R14.2
- net J1-3_5V: now also R16.1, U11.5 (I4); no longer U7.7 (I2)
- net at R9.2: now also U6.23 (PD3)
- net at R13.2: now also J1.1 (Pin_1); no longer U7.8 (I1)
- net J1-1_5V: now reaches R8.2
- net J1-1_5V: now also R13.1, U11.6 (I3); no longer U7.9 (I0)
- net Test_{4}: now reaches U6.1 (PA5)
- net Test_{4}: now also U2.1 (COM), J5.9 (Pin_9)
- net Test_{5}: now reaches U6.2 (PA6)
- net Test_{5}: now also U5.1 (COM), J5.11 (Pin_11)
- net at U6.27 (PD7): now also R20.1, SW1.1
- net RTS: now reaches U6.28 (PE0)
- net RTS: now also U12.3 (RTS)
- net CTS: now reaches U6.29 (PE1)
- net CTS: now also U12.11 (CTS)
- net Test_{6}: now reaches U6.3 (PA7)
- net Test_{6}: now also U4.1 (COM), J5.13 (Pin_13)
- net PDI_DATA: now reaches U6.34 (PDI_DATA)
- net PDI_DATA: now also J4.1 (Pin_1)
- net PDI_CLK: now reaches U6.35 (~{RESET}/PDI_CLK)
- net PDI_CLK: now also J4.5 (Pin_5)
- net at U6.37 (PR1/XTAL1): now also U13.3 (OUT)
- net +3.3VA: now reaches U6.4 (AREFB/PB0)
- net +3.3VA: now also U6.39 (AVCC), U6.40 (AREFA/PA0), C24.1, FB1.1
- net Test_{0}: now reaches U6.41 (PA1)
- net Test_{0}: now also U8.1 (COM), J5.1 (Pin_1)
- net Test_{1}: now reaches U6.42 (PA2)
- net Test_{1}: now also U10.1 (COM), J5.3 (Pin_3)
- net Test_{2}: now reaches U6.43 (PA3)
- net Test_{2}: now also U9.1 (COM), J5.5 (Pin_5)
- net Test_{3}: now reaches U6.44 (PA4)
- net Test_{3}: now also U7.1 (COM), J5.7 (Pin_7)
- net Test_{7}: now reaches U6.5 (PB1)
- net Test_{7}: now also U1.1 (COM), J5.15 (Pin_15)
- net Test_{Power}: now reaches U6.6 (PB2)
- net Test_{Power}: now also J5.17 (Pin_17), U11.1 (COM)
- removed net J1-7_2.5V_Test: R3.1, U4.16 (I15)
- removed net Test: U1.1 (COM), U10.1 (COM), U2.1 (COM), U4.1 (COM), U5.1 (COM), U7.1 (COM), U8.1 (COM), U9.1 (COM)
- new net: J1.7 (Pin_7), R3.2
- new net: J1.9 (Pin_9), R4.2
- new net: J1.13 (Pin_13), R6.2
- new net: J3.2 (Pin_2), R21.1
- new net: J3.4 (Pin_4), R22.1
- new net: J3.6 (Pin_6), R23.1
- new net: C19.1, U12.17 (3V3OUT)
- new net: J1.5 (Pin_5), R18.2
- new net: C22.1, J2.6 (Shield), R19.2
- new net: C20.1, J2.3 (D+), U12.15 (USBD+)
- new net: C21.1, J2.2 (D-), U12.16 (USBD-)
- new net: D6.2 (A), R15.1
- new net: J1.11 (Pin_11), R5.2
- new net: J1.3 (Pin_3), R16.2
- new net: J1.4 (Pin_4), R1.1
- new net: J1.6 (Pin_6), R2.1
- new net J1-5_5V: R17.2, R18.1, U11.4 (I5)
- new net VBUS: C14.1, J2.1 (VBUS), L1.1
- no-connect marks 16 -> 48
Other:
- note removed: "1. Start by measuring the rails 2. Loop through channels 1 by 1 in Sync with TestClock 3. Does not test pin-for-pin 5V or GND! Use manual inspection on individual pins."
- note removed: "NB: Test must go to analog capable pin. Can be split to two pins: analog and digital."
- note removed: "NB: UART?"
- moved on the sheet: C1, C10, C11, C12, C2, C3, C4, C5, C6, C7, C8, C9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
